File: keyboard.kicad_pcb (KiCad board)
At the start: 2 copper layers, 285 x 94.6 mm, 338 parts, among them IC1 ATMEGA32U4, J1 MINI, P1 CONN_1, P10 CONN_1, P11 CONN_1, P12 CONN_1, P13 CONN_1, P14 CONN_1, P15 CONN_1, P16 CONN_1, P17 CONN_1, P18 CONN_1, P19 CONN_1, P2 CONN_1, P20 CONN_1, P21 CONN_1, P22 CONN_1, P23 CONN_1, P24 CONN_1, P25 CONN_1, P26 CONN_1, P27 CONN_1, P28 CONN_1, P29 CONN_1, P3 CONN_1, P30 CONN_1, P31 CONN_1, P32 CONN_1, P33 CONN_1, P34 CONN_1, P35 CONN_1, P36 CONN_1, P37 CONN_1, P38 CONN_1, P39 CONN_1, P4 CONN_1, P40 CONN_1, P41 CONN_1, P42 CONN_1, P5 CONN_1, P6 CONN_1, P7 CONN_1, P8 CONN_1, P9 CONN_1, X1 ASX3F

Commit message: assign footprints.
Parts:
- DB05, DB051, DB10, DB101, DB102, DB15, DB151, DB55, DB551, DF21, DF211, DF22, DF221, DF23, DF231, DF232: value LEDa -> LED; footprint MX1A-led -> mx1a:MX1A-led
- DC3: footprint MX1A-ledlock -> mx1a:MX1A-led
- P1, P10, P11, P12, P13, P14, P15, P16, P17, P18, P19, P2, P20, P21, P22, P23, P24, P25, P26, P27, P28, P29, P3, P30, P31, P32, P33, P34, P35, P36, P37, P38, P39, P4, P40, P41, P42, P5, P6, P7, P8, P9: footprint pad -> pad:pad
- S031, S041, S0512, S09, S101, S102, S151, S301, S302, S50, S552, S601, S602, S63, S641, S6512, S661, S682, S691, S692, S7012: value MX1Aa -> MX1A
Connections:
- net /Matrix/CAPS_LED renamed /MOSI
- net /Matrix/col1 renamed /col1
- net /Matrix/col10 renamed /col10
- net /Matrix/col11 renamed /col11
- net /Matrix/col12 renamed /col12
- net /Matrix/col13 renamed /col13
- net /Matrix/col14 renamed /MISO
- net /Matrix/col2 renamed /col2
- net /Matrix/col3 renamed /col3
- net /Matrix/col4 renamed /col4
- net /Matrix/col5 renamed /col5
- net /Matrix/col6 renamed /col6
- net /Matrix/col7 renamed /col7
- net /Matrix/col8 renamed /SCK
- net /Matrix/col9 renamed /col9
- net /Matrix/row1 renamed /row1
- net /Matrix/row2 renamed /row2
- net /Matrix/row3 renamed /row3
- net /Matrix/row4 renamed /row4
- net /Matrix/row5 renamed /row5
- DC1 pad 2: N-000133 -> Net-(DC1-Pad2)
- DC2 pad 2: N-000133 -> Net-(DC1-Pad2)
- DF23 pad 2: N-000041 -> Net-(DF23-Pad2)
- DF231 pad 2: N-000041 -> Net-(DF23-Pad2)
- IC1 pad 42: (no net) -> Net-(IC1-Pad42)
- IC1 pad 8: (no net) -> Net-(IC1-Pad8)
- J1 pad 4: (no net) -> Net-(J1-Pad4)
- R15 pad 2: N-000041 -> Net-(DF23-Pad2)
- R4 pad 1: N-000133 -> Net-(DC1-Pad2)
- S0 pad 2: (no net) -> Net-(S0-Pad2)
- S0 pad 4: (no net) -> Net-(S0-Pad4)
Routing:
- net Net-(DC1-Pad2): track 0.00 -> 35.0 mm, vias 0 -> 1
- net N-000133: track 35.0 -> 0.00 mm, vias 1 -> 0
- net Net-(DF23-Pad2): track 0.00 -> 20.3 mm
- net N-000041: track 20.3 -> 0.00 mm
