File: leds.sch (KiCad schematic (older format))
At the start: 66 parts

Commit message: remap symbols.
Parts:
- DB02, DB04, DB041, DB05, DB051, DB06, DB07, DB09, DB10, DB101, DB102, DB11, DB14, DB15, DB151, DB16, DB17, DB19, DB21, DB22, DB23, DB24, DB26, DB27, DB28, DB29, DB30, DB301, DB302, DB31, DB32, DB33, DB34, DB36, DB37, DB38, DB39, DB41, DB42, DB43, DB44, DB46, DB47, DB48, DB49, DB50, DB51, DB52, DB53, DB54, DB55, DB551, DB56, DB57, DB58, DB59, DB61, DB62, DB63, DB66, DB661, DB67, DB68, DB681, DB682, DB69: symbol LED -> device:LED
Changed lines of the file:
@@
-EESchema Schematic File Version 2
-LIBS:power
-LIBS:mx1a-simple
-LIBS:aker
-LIBS:atmega32u4
-LIBS:dtsjw
-LIBS:oupiin_usb
-LIBS:device
-LIBS:conn
-LIBS:keyboard-cache
-EELAYER 25 0
+EESchema Schematic File Version 4
+EELAYER 29 0
 EELAYER END
 $Descr A4 11693 8268
@@
 $EndDescr
 $Comp
-L LED DB21
+L device:LED DB21
 U 1 1 51900721
 P 4450 1950
@@
 $EndComp
 $Comp
-L LED DB26
+L device:LED DB26
 U 1 1 51900730
 P 5000 1950
@@
 $EndComp
 $Comp
-L LED DB31
+L device:LED DB31
 U 1 1 51900737
 P 5550 1950
@@
 $EndComp
 $Comp
-L LED DB36
+L device:LED DB36
 U 1 1 5190073E
 P 6100 1950
@@
 $EndComp
 $Comp
-L LED DB06
+L device:LED DB06
 U 1 1 5190074C
 P 2800 1950
@@
 $EndComp
 $Comp
-L LED DB11
+L device:LED DB11
 U 1 1 51900753
 P 3350 1950
@@
 $EndComp
 $Comp
-L LED DB16
+L device:LED DB16
 U 1 1 5190075A
 P 3900 1950
@@
 $EndComp
 $Comp
-L LED DB61
+L device:LED DB61
 U 1 1 51900761
 P 8850 1950
@@
 $EndComp
 $Comp
-L LED DB66
+L device:LED DB66
 U 1 1 51900768
 P 9400 1950
@@
 $EndComp
 $Comp
-L LED DB41
+L device:LED DB41
 U 1 1 5190077D
 P 6650 1950
@@
 $EndComp
 $Comp
-L LED DB46
+L device:LED DB46
 U 1 1 51900784
 P 7200 1950
@@
 $EndComp
 $Comp
-L LED DB51
+L device:LED DB51
 U 1 1 5190078B
 P 7750 1950
@@
 $EndComp
 $Comp
-L LED DB56
+L device:LED DB56
 U 1 1 51900792
 P 8300 1950
@@
 $EndComp
 $Comp
-L LED DB22
+L device:LED DB22
 U 1 1 51900799
 P 4450 2850
@@
 $EndComp
 $Comp
-L LED DB27
+L device:LED DB27
 U 1 1 519007A0
 P 5000 2850
@@
 $EndComp
 $Comp
-L LED DB32
+L device:LED DB32
 U 1 1 519007A7
 P 5550 2850
@@
 $EndComp
 $Comp
-L LED DB37
+L device:LED DB37
 U 1 1 519007AE
 P 6100 2850
@@
 $EndComp
 $Comp
-L LED DB02
+L device:LED DB02
 U 1 1 519007B5
 P 2250 2850
@@
 $EndComp
 $Comp
-L LED DB07
+L device:LED DB07
 U 1 1 519007BC
 P 2800 2850
@@
 $EndComp
 $Comp
-L LED DB17
+L device:LED DB17
 U 1 1 519007CA
 P 3900 2850
@@
 $EndComp
 $Comp
-L LED DB62
+L device:LED DB62
 U 1 1 519007D1
 P 8850 2850
@@
 $EndComp
 $Comp
-L LED DB67
+L device:LED DB67
 U 1 1 519007D8
 P 9400 2850
@@
 $EndComp
 $Comp
-L LED DB42
+L device:LED DB42
 U 1 1 519007E6
 P 6650 2850
@@
 $EndComp
 $Comp
-L LED DB47
+L device:LED DB47
 U 1 1 519007ED
 P 7200 2850
@@
 $EndComp
 $Comp
-L LED DB52
+L device:LED DB52
 U 1 1 519007F4
 P 7750 2850
@@
 $EndComp
 $Comp
-L LED DB57
+L device:LED DB57
 U 1 1 519007FB
 P 8300 2850
@@
 $EndComp
 $Comp
-L LED DB23
+L device:LED DB23
 U 1 1 51900802
 P 4450 3500
@@
 $EndComp
 $Comp
-L LED DB28
+L device:LED DB28
 U 1 1 51900809
 P 5000 3500
@@
 $EndComp
 $Comp
-L LED DB33
+L device:LED DB33
 U 1 1 51900810
 P 5550 3500
@@
 $EndComp
 $Comp
-L LED DB38
+L device:LED DB38
 U 1 1 51900817
 P 6100 3500
@@
 $EndComp
 $Comp
-L LED DB63
+L device:LED DB63
 U 1 1 5190083A
 P 8850 3500
@@
 $EndComp
 $Comp
-L LED DB68
+L device:LED DB68
 U 1 1 51900841
 P 9400 3500
@@
 $EndComp
 $Comp
-L LED DB43
+L device:LED DB43
 U 1 1 5190084F
 P 6650 3500
@@
 $EndComp
 $Comp
-L LED DB48
+L device:LED DB48
 U 1 1 51900856
 P 7200 3500
@@
 $EndComp
 $Comp
-L LED DB53
+L device:LED DB53
 U 1 1 5190085D
 P 7750 3500
@@
 $EndComp
 $Comp
-L LED DB58
+L device:LED DB58
 U 1 1 51900864
 P 8300 3500
@@
 $EndComp
 $Comp
-L LED DB24
+L device:LED DB24
 U 1 1 5190086B
 P 4450 4650
@@
 $EndComp
 $Comp
-L LED DB29
+L device:LED DB29
 U 1 1 51900872
 P 5000 4650
@@
 $EndComp
 $Comp
-L LED DB34
+L device:LED DB34
 U 1 1 51900879
 P 5550 4650
@@
 $EndComp
 $Comp
-L LED DB39
+L device:LED DB39
 U 1 1 51900880
 P 6100 4650
@@
 $EndComp
 $Comp
-L LED DB04
+L device:LED DB04
 U 1 1 51900887
 P 2250 4650
@@
 $EndComp
 $Comp
-L LED DB09
+L device:LED DB09
 U 1 1 5190088E
 P 2800 4650
@@
 $EndComp
 $Comp
-L LED DB14
+L device:LED DB14
 U 1 1 51900895
 P 3350 4650
@@
 $EndComp
 $Comp
-L LED DB19
+L device:LED DB19
 U 1 1 5190089C
 P 3900 4650
@@
 $EndComp
 $Comp
-L LED DB44
+L device:LED DB44
 U 1 1 519008B8
 P 6650 4650
@@
 $EndComp
 $Comp
-L LED DB49
+L device:LED DB49
 U 1 1 519008BF
 P 7200 4650
@@
 $EndComp
 $Comp
-L LED DB54
+L device:LED DB54
 U 1 1 519008C6
 P 7750 4650
@@
 $EndComp
 $Comp
-L LED DB59
+L device:LED DB59
 U 1 1 519008CD
 P 8300 4650
@@
 $EndComp
 $Comp
-L LED DB05
+L device:LED DB05
 U 1 1 519008F0
 P 2250 5550
@@
 $EndComp
 $Comp
-L LED DB10
+L device:LED DB10
 U 1 1 519008F7
 P 2800 5550
@@
 $EndComp
 $Comp
-L LED DB15
+L device:LED DB15
 U 1 1 519008FE
 P 3350 5550
@@
 $EndComp
 $Comp
-L LED DB50
+L device:LED DB50
 U 1 1 51900928
 P 7200 5550
@@
 $EndComp
 $Comp
-L LED DB55
+L device:LED DB55
 U 1 1 5190092F
 P 7750 5550
@@
 $EndComp
 $Comp
-L LED DB30
+L device:LED DB30
 U 1 1 519008DB
 P 5000 5550
@@
 $EndComp
 $Comp
-L LED DB551
+L device:LED DB551
 U 1 1 51C02CCF
 P 7750 5800
@@
 $EndComp
 $Comp
-L LED DB301
+L device:LED DB301
 U 1 1 51C0300D
 P 5000 5800
@@
 $EndComp
 $Comp
-L LED DB302
+L device:LED DB302
 U 1 1 51C03013
 P 5000 6050
@@
 $EndComp
 $Comp
-L LED DB051
+L device:LED DB051
 U 1 1 51C0378E
 P 2250 5800
@@
 $EndComp
 $Comp
-L LED DB101
+L device:LED DB101
 U 1 1 51C065B4
 P 2800 5800
@@
 $EndComp
 $Comp
-L LED DB102
+L device:LED DB102
 U 1 1 51C065BA
 P 2800 6050
@@
 $EndComp
 $Comp
-L LED DB151
+L device:LED DB151
 U 1 1 51C06955
 P 3350 5800
@@
 esc
 $Comp
-L LED DB69
+L device:LED DB69
 U 1 1 51C41A1A
 P 9400 4650
@@
 Fn
 $Comp
-L LED DB041
+L device:LED DB041
 U 1 1 51D98243
 P 2250 4900
@@
 Connection ~ 2050 4900
 $Comp
-L LED DB661
+L device:LED DB661
 U 1 1 51D9840C
 P 9400 2200
@@
 Connection ~ 9200 2200
 $Comp
-L LED DB681
+L device:LED DB681
 U 1 1 51D988E8
 P 9400 3750
@@
 $EndComp
 $Comp
-L LED DB682
+L device:LED DB682
 U 1 1 51D988EE
 P 9400 4000

Commit message: assign footprints.
Parts:
- DB05, DB051, DB10, DB101, DB102, DB15, DB151, DB55, DB551: footprint (none) -> mx1a:MX1A-led
Connections:
- wire segments 74 -> 206
